Commit message: .

File: install/crane_simulator/share/crane_simulator/crane.urdf (robot description, URDF)
Before this commit: robot crane, 2 links, 1 joints
Links:
- added link toolpoint; visual box size=0 0 0
Joints:
- added joint crane_boom_to_toolpoint: type fixed, parent crane_boom, child toolpoint, origin xyz=3.6 0 0 rpy=0 0 0

File: install/crane_visualization/share/crane_visualization/urdf/green_crane.urdf (robot description, URDF)
Before this commit: robot green_crane, 2 links, 1 joints
Links:
- added link toolpoint; visual box size=0 0 0
Joints:
- added joint crane_boom_to_toolpoint: type fixed, parent crane_boom, child toolpoint, origin xyz=3.6 0 0 rpy=0 0 0

File: install/crane_visualization/share/crane_visualization/urdf/simple_green_crane.urdf (robot description, URDF)
Before this commit: robot simple_green_crane, 2 links, 1 joints
Links:
- added link toolpoint; visual box size=0 0 0
Joints:
- added joint crane_boom_to_toolpoint: type fixed, parent crane_boom, child toolpoint, origin xyz=3.6 0 0 rpy=0 0 0

File: src/crane_visualization/urdf/simple_green_crane.urdf (robot description, URDF)
Before this commit: robot simple_green_crane, 2 links, 1 joints
Links:
- added link toolpoint; visual box size=0 0 0
Joints:
- added joint crane_boom_to_toolpoint: type fixed, parent crane_boom, child toolpoint, origin xyz=3.6 0 0 rpy=0 0 0
